File: Acorn-Electron/Cumana-Disk-Interface/Cumana-Disk-Interface.sch (KiCad schematic (older format))
At the start: 54 parts, among them J1 Bottom Top, J2 CONN_12X2, J3 Conn_01x34_Female, Q2 Q_NPN_CBE, Q3 Q_NPN_CBE, Q4 Q_PNP_CBE, Q5 Q_NPN_CBE, U1 74LS138, U10 74LS174, U11 M5W1793-02P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

Commit message: Cumana disk interface schematic update and pdf
Parts:
- A1, A2, A3, A4, A5, A6, A7, C2, C3: symbol Cumana-Electron-Disk-Interface:C -> Cumana-Disk-Interface:C
- C1, C4: symbol Cumana-Electron-Disk-Interface:CP1 -> Cumana-Disk-Interface:CP1
- D1, D2: symbol Cumana-Electron-Disk-Interface:Diode -> Cumana-Disk-Interface:Diode
- D3: symbol Cumana-Electron-Disk-Interface:D_Zener -> Cumana-Disk-Interface:D_Zener
- J1: symbol Cumana-Electron-Disk-Interface:CONN_9X2 -> Cumana-Disk-Interface:CONN_9X2
- J2: symbol Cumana-Electron-Disk-Interface:CONN_12X2 -> Cumana-Disk-Interface:CONN_12X2
- J3: symbol Cumana-Electron-Disk-Interface:Conn_01x34_Female -> Cumana-Disk-Interface:Conn_01x34_Female
- Q2, Q3, Q5: symbol Cumana-Electron-Disk-Interface:Q_NPN_CBE -> Cumana-Disk-Interface:Q_NPN_CBE
- Q4: symbol Cumana-Electron-Disk-Interface:Q_PNP_CBE -> Cumana-Disk-Interface:Q_PNP_CBE
- R1, R12, R13, R14, R15, R17, R18, R19, R2, R20, R3, R4, R5, R6, R7, R8, R9: symbol Cumana-Electron-Disk-Interface:R -> Cumana-Disk-Interface:R
- U1: symbol Cumana-Electron-Disk-Interface:74LS138 -> Cumana-Disk-Interface:74LS138
- U10: symbol Cumana-Electron-Disk-Interface:74LS174 -> Cumana-Disk-Interface:74LS174
- U11: symbol Cumana-Electron-Disk-Interface:M5W1793-02P -> Cumana-Disk-Interface:M5W1793-02P
- U12: symbol Cumana-Electron-Disk-Interface:74LS161 -> Cumana-Disk-Interface:74LS161
- U13: symbol Cumana-Electron-Disk-Interface:FDC9216B -> Cumana-Disk-Interface:FDC9216B
- U14: symbol Cumana-Electron-Disk-Interface:7406 -> Cumana-Disk-Interface:7406
- U2: symbol Cumana-Electron-Disk-Interface:74LS00 -> Cumana-Disk-Interface:74LS00
- U3: symbol Cumana-Electron-Disk-Interface:74LS02 -> Cumana-Disk-Interface:74LS02
- U4, U5: symbol Cumana-Electron-Disk-Interface:27128 -> Cumana-Disk-Interface:27128
- U6: symbol Cumana-Electron-Disk-Interface:CDM6116 -> Cumana-Disk-Interface:CDM6116
- U7: symbol Cumana-Electron-Disk-Interface:HD146818 -> Cumana-Disk-Interface:HD146818
- U8: symbol Cumana-Electron-Disk-Interface:74LS32 -> Cumana-Disk-Interface:74LS32
- U9: symbol Cumana-Electron-Disk-Interface:74LS04 -> Cumana-Disk-Interface:74LS04
- VC1: symbol Cumana-Electron-Disk-Interface:C_Variable -> Cumana-Disk-Interface:C_Variable
- Y1: symbol Cumana-Electron-Disk-Interface:Crystal_Small -> Cumana-Disk-Interface:Crystal_Small
