File: Acorn-Electron/Cumana-Disk-Interface/Cumana-Disk-Interface.kicad_pcb (KiCad board)
At the start: 2 copper layers, 148 x 118.7 mm, 55 parts, among them J1 Bottom Top, J2 CONN_12X2, J3 Conn_01x34_Female, Q2 Q_NPN_CBE, Q3 Q_NPN_CBE, Q4 Q_PNP_CBE, Q5 Q_NPN_CBE, U1 74LS138, U10 74LS174, U11 M5W1793-02P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

Commit message: upgraded to KiCad 6.0
Other:
- net class Default removed
